File: PCB/ESP32-DualCAN.kicad_sch (KiCad schematic)
At the start: 31 parts, among them J1 Molex 70553 6p, J2 Conn_01x10_Socket, J3 Conn_01x10_Socket, J4 holes, J5 pads, J6 holes, J7 pads, U1 LV2862Y, U2 ESP32-C6-SuperMini, U3 TCAN1044AV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

Commit message: /PCB folder
Parts:
- D3: LCSC DSK38 -> C28646291
Changed lines of the file:
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@@
 			)
 		)
-		(property "LCSC" "DSK38"
+		(property "LCSC" "C28646291"
 			(at 71.4375 17.145 0)
 			(effects
