File: hardware/ESP32-DualCAN.kicad_sch (KiCad schematic)
At the start: 35 parts, among them J1 Molex 70553 6p, J2 Conn_01x10_Socket, J3 Conn_01x10_Socket, J4 holes, J5 pads, J6 holes, J7 pads, U1 LV2862Y, U2 ESP32-C6-SuperMini, U3 TCAN1044AV, U4 TCAN1044AV, U5 ESP32-C6-Zero, U6 ESP32-C6-SuperMini

Commit message: DCDC load test
Parts:
- U1: value LV2862Y -> MLMR16006Y; Alternative LV2862Y, LMR16006Y, LMR51606YF -> LV2862Y, LMR16006Y, LMR51606YF, MLMR16006Y
Other:
- note added: "Tested 0.5A max continuous accross 9-60V at 22C ambient before thermal shutdown"
Changed lines of the file:
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@@
 		)
 	)
+	(text "Tested 0.5A max continuous accross 9-60V at 22C ambient\nbefore thermal shutdown"
+		(exclude_from_sim no)
+		(at 78.232 46.736 0)
+		(effects
+			(font
+				(size 1.27 1.27)
+			)
+			(justify left top)
+		)
+	)
 	(text "ESP32-C6-SuperMini also can be attached using pin headers.\nNote, the pin config would need to be changed in the firmware"
 		(exclude_from_sim no)
@@
 			)
 		)
-		(property "Value" "LV2862Y"
+		(property "Value" "MLMR16006Y"
 			(at 139.7 22.098 0)
 			(show_name no)
@@
 			)
 		)
-		(property "Datasheet" "https://www.ti.com/lit/ds/symlink/lv2862.pdf"
+		(property "Datasheet" "https://www.lcsc.com/datasheet/C42403103.pdf"
 			(at 137.16 26.67 0)
 			(hide yes)
@@
 			)
 		)
-		(property "Alternative" "LV2862Y, LMR16006Y, LMR51606YF"
+		(property "Alternative" "LV2862Y, LMR16006Y, LMR51606YF, MLMR16006Y"
 			(at 139.7 29.21 0)
 			(hide yes)

Commit message: MLMR16006Y needs pull up on enable pin
Connections:
- net BATT_Diode: now also U1.4 (EN)
- no-connect marks 2 -> 1
Changed lines of the file:
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@@
+	)
+	(junction
+		(at 128.27 26.67)
+		(diameter 0)
+		(color 0 0 0 0)
 	)
 	(junction
@@
 		(at 157.48 107.95)
 	)
-	(no_connect
-		(at 129.54 31.75)
-	)
 	(wire
 		(pts
@@
 	(wire
 		(pts
+			(xy 128.27 31.75) (xy 129.54 31.75)
+		)
+		(stroke
+			(width 0)
+			(type default)
+		)
+	)
+	(wire
+		(pts
 			(xy 45.72 179.07) (xy 50.8 179.07)
 		)
@@
 	(wire
 		(pts
+			(xy 128.27 26.67) (xy 128.27 31.75)
+		)
+		(stroke
+			(width 0)
+			(type default)
+		)
+	)
+	(wire
+		(pts
 			(xy 198.12 246.38) (xy 209.55 246.38)
 		)
@@
 	(wire
 		(pts
-			(xy 115.57 26.67) (xy 129.54 26.67)
+			(xy 115.57 26.67) (xy 128.27 26.67)
 		)
 		(stroke
@@
 		)
 		(stroke
+			(width 0)
+			(type default)
+		)
+	)
+	(wire
+		(pts
+			(xy 128.27 26.67) (xy 129.54 26.67)
+		)
+		(stroke
